File: transistor-amp.kicad_pcb (KiCad board)
At the start: 2 copper layers, 47.5 x 50.5 mm, 24 parts, among them J1 Conn_01x06_Pin, Q1 PNP, Q10 NPN, Q2 PNP, Q3 NPN, Q4 NPN, Q5 NPN, Q6 PNP, Q7 PNP, Q8 PNP, Q9 NPN

Commit message: add gerber/drill files
Parts:
- removed the Q1 at (81.5, 82.5)
- added R1: 10k, Resistor_THT:R_Axial_DIN0207_L6.3mm_D2.5mm_P7.62mm_Horizontal, F.Cu at (83.0, 87.3)
- R2: renamed from R3; value 30k -> 10k
- RV1: value R_Potentiometer_US -> 10k
- renumbered D2 to D1, D1 to D2, Q2 to Q1, Q3 to Q2, Q4 to Q3, Q6 to Q4, Q7 to Q5, Q5 to Q6, Q8 to Q7, Q10 to Q8, R1 to R3, R2 to R5, R7 to R6, R6 to R7, R5 to R8
Connections:
- net /AUDIO_IN renamed Net-(J1-Pin_1)
- Q1 pad 3: Net-(Q2-E) -> Net-(Q1-E)
- Q2 pad 1: Net-(Q2-E) -> Net-(Q1-E)
- Q2 pad 2: Net-(Q3-B) -> Net-(Q1-E)
- Q3 pad 2: Net-(Q3-B) -> Net-(Q1-E)
Routing:
- net Net-(Q1-E): track 0.00 -> 17.4 mm
- net Net-(Q2-E): track 8.64 -> 0.00 mm
- net Net-(Q3-B): track 7.45 -> 0.00 mm
- net GND: track 0.00 -> 5.48 mm
- net Net-(Q1-B): track 9.53 -> 8.38 mm
Other:
- board text added: "Volume"
