File: transistor-amp.kicad_sch (KiCad schematic)
At the start: 24 parts, among them J1 Conn_01x06_Pin, Q1 PNP, Q10 NPN, Q2 PNP, Q3 NPN, Q4 NPN, Q5 NPN, Q6 PNP, Q7 PNP, Q8 PNP, Q9 NPN

Commit message: add gerber/drill files
Parts:
- removed Q1: PNP, Package_TO_SOT_THT:TO-92L_Inline, symbol Simulation_SPICE:PNP
- added R1: 10k, Resistor_THT:R_Axial_DIN0207_L6.3mm_D2.5mm_P7.62mm_Horizontal, symbol Device:R_US
- R2: renamed from R3; value 30k -> 10k
- RV1: value R_Potentiometer_US -> 10k
- renumbered D2 to D1, D1 to D2, Q2 to Q1, Q3 to Q2, Q4 to Q3, Q6 to Q4, Q7 to Q5, Q5 to Q6, Q8 to Q7, Q10 to Q8, R1 to R3, R2 to R5, R7 to R6, R6 to R7, R5 to R8
Connections:
- net GND: now also R1.2
- net at Q1.3 (E), Q2.1 (C): now also Q2.2 (B), Q3.2 (B)
- net at Q1.2 (B): now also R1.1
- net AUDIO_IN: no longer names the net of J1.1 (Pin_1), RV1.1
Other:
- moved on the sheet: BT1, BT2, J1, RV1
